File: SolderSolar_PCB/SolderSolar.sch (KiCad schematic (older format))
At the start: 14 parts, among them P1 SOLAR_V, P2 LOGO1, P3 LOGO2, P4 PCB, P5 LOGO3, SW1 RED, SW2 WHITE

Commit message: Updated PCB for KiCAD
Parts:
- C1: symbol CP -> Device:CP
- D1: symbol D_Schottky -> Device:D_Schottky
- D2, D3: symbol LED-RESCUE-SolderSolar2017 -> SolderSolar-rescue:LED-RESCUE-SolderSolar2017
- P1: symbol CONN_01X02 -> conn:CONN_01X02
- P2, P3, P4, P5: symbol CONN_01X01 -> conn:CONN_01X01
- R1, R2: symbol R -> Device:R
- SC1: symbol Solar_Cells -> Device:Solar_Cells
- SW1, SW2: symbol SW_PUSH -> SolderSolar-rescue:SW_PUSH
Changed lines of the file:
@@
-EESchema Schematic File Version 2
-LIBS:SolderSolar2017-rescue
-LIBS:power
-LIBS:device
-LIBS:transistors
-LIBS:conn
-LIBS:linear
-LIBS:regul
-LIBS:74xx
-LIBS:cmos4000
-LIBS:adc-dac
-LIBS:memory
-LIBS:xilinx
-LIBS:microcontrollers
-LIBS:dsp
-LIBS:microchip
-LIBS:analog_switches
-LIBS:motorola
-LIBS:texas
-LIBS:intel
-LIBS:audio
-LIBS:interface
-LIBS:digital-audio
-LIBS:philips
-LIBS:display
-LIBS:cypress
-LIBS:siliconi
-LIBS:opto
-LIBS:atmel
-LIBS:contrib
-LIBS:valves
-LIBS:matts_components
-LIBS:SolderSolar2017-cache
-EELAYER 25 0
+EESchema Schematic File Version 4
+EELAYER 30 0
 EELAYER END
 $Descr A4 11693 8268
@@
 $EndDescr
 $Comp
-L LED-RESCUE-SolderSolar2017 D2
+L SolderSolar-rescue:LED-RESCUE-SolderSolar2017 D2
 U 1 1 58A49D8B
 P 7450 3400
@@
 $EndComp
 $Comp
-L LED-RESCUE-SolderSolar2017 D3
+L SolderSolar-rescue:LED-RESCUE-SolderSolar2017 D3
 U 1 1 58A49DE6
 P 7450 3800
@@
 $EndComp
 $Comp
-L CP C1
+L Device:CP C1
 U 1 1 58A49EA0
 P 5000 3850
@@
 $EndComp
 $Comp
-L Solar_Cells SC1
+L Device:Solar_Cells SC1
 U 1 1 58A49F68
 P 3950 3850
@@
 $EndComp
 $Comp
-L R R1
+L Device:R R1
 U 1 1 58A49FAD
 P 6900 3400
@@
 $EndComp
 $Comp
-L R R2
+L Device:R R2
 U 1 1 58A4A023
 P 6900 3800
@@
 $EndComp
 $Comp
-L D_Schottky D1
+L Device:D_Schottky D1
 U 1 1 58A4A198
 P 4400 3400
@@
 $EndComp
 $Comp
-L SW_PUSH SW1
+L SolderSolar-rescue:SW_PUSH SW1
 U 1 1 58A4A835
 P 6300 3400
@@
 $EndComp
 $Comp
-L SW_PUSH SW2
+L SolderSolar-rescue:SW_PUSH SW2
 U 1 1 58A4A8D6
 P 6300 3800
@@
 $EndComp
 $Comp
-L CONN_01X01 P4
+L conn:CONN_01X01 P4
 U 1 1 58A4A93E
 P 8450 3400
@@
 $EndComp
 $Comp
-L CONN_01X01 P2
+L conn:CONN_01X01 P2
 U 1 1 58A4A9B1
 P 8450 3750
@@
 $EndComp
 $Comp
-L CONN_01X01 P3
+L conn:CONN_01X01 P3
 U 1 1 58A4AA34
 P 8450 4050
@@
 $EndComp
 $Comp
-L GND #PWR01
+L power:GND #PWR01
 U 1 1 58A4AEF1
 P 5650 4250
@@
 	3950 3400 4250 3400
 Wire Wire Line
-	4550 3400 6000 3400
+	4550 3400 5000 3400
 Wire Wire Line
 	3950 4050 3950 4150
 Wire Wire Line
-	3950 4150 7800 4150
-Wire Wire Line
-	7800 4150 7800 3400
+	3950 4150 5000 4150
+Wire Wire Line
+	7800 4150 7800 3800
 Wire Wire Line
 	7800 3400 7600 3400
@@
 Resistor Calculations:\nRED - Vinput minimum 3V Maximum 5V\nNeeds 5mA to run at 1.8V\nSo V=IR \n3-1.8 = 0.005 x R, R = 240\n5-1.8 = 0.005 x R, R = 640\nUse 330R\n\nWHITE\nNeeds 5mA to run at 2.6V\nSo V=IR \n3-2.6 = 0.005 x R, R = 80\n5-2.6 = 0.005 x R, R = 480\nUse 120R\n
 $Comp
-L CONN_01X02 P1
+L conn:CONN_01X02 P1
 U 1 1 58B44224
 P 5850 2950
@@
 Connection ~ 5300 3400
 $Comp
-L CONN_01X01 P5
+L conn:CONN_01X01 P5
 U 1 1 58C13779
 P 8450 4350
@@
 $EndComp
 NoConn ~ 8250 4350
+Wire Wire Line
+	7800 3800 7800 3400
+Wire Wire Line
+	5750 3400 6000 3400
+Wire Wire Line
+	5000 3400 5300 3400
+Wire Wire Line
+	5000 4150 5400 4150
+Wire Wire Line
+	5650 4150 7800 4150
+Wire Wire Line
+	5400 4150 5650 4150
+Wire Wire Line
+	5300 3400 5750 3400
 $EndSCHEMATC
