File: SolderSolar_PCB/SolderSolar.kicad_sch (KiCad schematic)
At the start: 13 parts, among them P2 LOGO1, P3 LOGO2, P4 PCB, P5 LOGO3, SW1 RED, SW2 WHITE

Commit message: Updated with new logo and instructions on PCB
Parts:
- C1: footprint REInnovationFootprint:C_0_47F_SuperCap -> REInnovationFootprint:C_0_47F_SuperCap_3POS
- P2: footprint CuriousElectric3:CEC_Globe_10mm_FCU -> CuriousElectric3:2019_011_16_CuriousElectricCompany_Logo_Round_Logo_No_words_KiCAD_10mm_PCBLogo
- P4: footprint REInnovationFootprint:PV_50x30mmEdgeCut -> (none)

Commit message: changed hole size for production
Parts:
- SC1: footprint REInnovationFootprint:PV_50x30mm_NoOutline -> REInnovationFootprint:PV_50x30mm_NoOutline_v2
Changed lines of the file:
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@@
 			)
 		)
-		(property "Footprint" "REInnovationFootprint:PV_50x30mm_NoOutline"
+		(property "Footprint" "REInnovationFootprint:PV_50x30mm_NoOutline_v2"
 			(at 100.33 96.266 90)
 			(effects
